File: hardware/Ponto.sch (KiCad schematic (older format))
At the start: 9 parts, among them P1 RFID-RC522-MODULE, P2 CONN_01X04, P3 USB_B, U1 ESP-07v2, U2 LM1117-3.3

Commit message: Começando PCB
Parts:
- added D3: LED, LEDs:LED-5MM, symbol LED
- added R3: 4K7, Resistors_THT:R_Axial_DIN0617_L17.0mm_D6.0mm_P20.32mm_Horizontal, symbol R
- P3: footprint (none) -> Connectors:USB_B
- R1, R2: footprint Resistors_Universal:Resistor_SMD+THTuniversal_0805to1206_RM10_HandSoldering -> Resistors_THT:R_Axial_DIN0617_L17.0mm_D6.0mm_P20.32mm_Horizontal
- U2: footprint TO_SOT_Packages_SMD:SOT-223 -> Common-Parts-Library:TO-220-3
Connections:
- wire segments 39 -> 48
- no-connect marks 8 -> 7
Other:
- moved on the sheet: P3
Changed lines of the file:
@@
 LIBS:tsop4856
 LIBS:usblc6-4
+LIBS:Ponto-cache
 EELAYER 25 0
 EELAYER END
@@
 F 0 "U2" H 7900 1500 50  0000 C CNN
 F 1 "LM1117-3.3" H 7800 2000 50  0000 C CNN
-F 2 "TO_SOT_Packages_SMD:SOT-223" H 7800 1750 50  0001 C CNN
+F 2 "Common-Parts-Library:TO-220-3" H 7800 1750 50  0001 C CNN
 F 3 "" H 7800 1750 50  0000 C CNN
 	1    7800 1750
@@
 F 0 "P3" H 9400 1500 50  0000 C CNN
 F 1 "USB_B" H 9150 1900 50  0000 C CNN
-F 2 "" V 9150 1600 50  0001 C CNN
+F 2 "Connectors:USB_B" V 9150 1600 50  0001 C CNN
 F 3 "" V 9150 1600 50  0000 C CNN
 	1    9200 1700
-	1    0    0    -1
+	0    1    1    0
 $EndComp
 $Comp
 L GND #PWR01
 U 1 1 59A457D0
-P 9300 2100
-F 0 "#PWR01" H 9300 1850 50  0001 C CNN
-F 1 "GND" H 9300 1950 50  0000 C CNN
-F 2 "" H 9300 2100 50  0000 C CNN
-F 3 "" H 9300 2100 50  0000 C CNN
-	1    9300 2100
+P 8750 1700
+F 0 "#PWR01" H 8750 1450 50  0001 C CNN
+F 1 "GND" H 8750 1550 50  0000 C CNN
+F 2 "" H 8750 1700 50  0000 C CNN
+F 3 "" H 8750 1700 50  0000 C CNN
+	1    8750 1700
 	1    0    0    -1
 $EndComp
@@
 F 0 "R1" V 7480 2950 50  0000 C CNN
 F 1 "4K7" V 7400 2950 50  0000 C CNN
-F 2 "Resistors_Universal:Resistor_SMD+THTuniversal_0805to1206_RM10_HandSoldering" V 7330 2950 50  0001 C CNN
+F 2 "Resistors_THT:R_Axial_DIN0617_L17.0mm_D6.0mm_P20.32mm_Horizontal" V 7330 2950 50  0001 C CNN
 F 3 "" H 7400 2950 50  0000 C CNN
 	1    7400 2950
@@
 F 0 "R2" V 7480 3250 50  0000 C CNN
 F 1 "4K7" V 7400 3250 50  0000 C CNN
-F 2 "Resistors_Universal:Resistor_SMD+THTuniversal_0805to1206_RM10_HandSoldering" V 7330 3250 50  0001 C CNN
+F 2 "Resistors_THT:R_Axial_DIN0617_L17.0mm_D6.0mm_P20.32mm_Horizontal" V 7330 3250 50  0001 C CNN
 F 3 "" H 7400 3250 50  0000 C CNN
 	1    7400 3250
@@
 Wire Wire Line
 	8100 1750 8450 1750
-Wire Wire Line
-	9500 2000 9500 1600
-Wire Wire Line
-	9300 2000 9500 2000
-NoConn ~ 6800 3450
 NoConn ~ 5000 3250
 NoConn ~ 5000 3150
@@
 Wire Wire Line
 	8750 2850 8700 2850
+$Comp
+L LED D3
+U 1 1 59A59BC3
+P 7800 3600
+F 0 "D3" H 7800 3700 50  0000 C CNN
+F 1 "LED" H 7800 3500 50  0000 C CNN
+F 2 "LEDs:LED-5MM" H 7800 3600 50  0001 C CNN
+F 3 "" H 7800 3600 50  0000 C CNN
+	1    7800 3600
+	-1   0    0    1
+$EndComp
+$Comp
+L R R3
+U 1 1 59A59C26
+P 7400 3600
+F 0 "R3" V 7480 3600 50  0000 C CNN
+F 1 "4K7" V 7400 3600 50  0000 C CNN
+F 2 "Resistors_THT:R_Axial_DIN0617_L17.0mm_D6.0mm_P20.32mm_Horizontal" V 7330 3600 50  0001 C CNN
+F 3 "" H 7400 3600 50  0000 C CNN
+	1    7400 3600
+	0    1    1    0
+$EndComp
+Wire Wire Line
+	6800 3450 7200 3450
+Wire Wire Line
+	7200 3450 7200 3600
+Wire Wire Line
+	7200 3600 7250 3600
+Wire Wire Line
+	7550 3600 7650 3600
+$Comp
+L GND #PWR012
+U 1 1 59A59CEA
+P 8200 3600
+F 0 "#PWR012" H 8200 3350 50  0001 C CNN
+F 1 "GND" H 8200 3450 50  0000 C CNN
+F 2 "" H 8200 3600 50  0000 C CNN
+F 3 "" H 8200 3600 50  0000 C CNN
+	1    8200 3600
+	1    0    0    -1
+$EndComp
+Wire Wire Line
+	7950 3600 8200 3600
+Wire Wire Line
+	8800 1700 8750 1700
+Wire Wire Line
+	8750 1700 8750 1600
+Wire Wire Line
+	8750 1600 8800 1600
+Wire Wire Line
+	9000 2000 9000 2100
+Wire Wire Line
+	9000 2100 9300 2100
+Wire Wire Line
+	9300 2000 9400 2000
 $EndSCHEMATC
